File: Hard/ModPrincipal/UARTAislada.sch (KiCad schematic (older format))
At the start: 1 part

Commit message: Agrego UART aislada y salidas digitales
Parts:
- added C? (x4): 100nF, Capacitor_SMD:C_0805_2012Metric_Pad1.15x1.40mm_HandSolder, symbol pspice:C
- added J? (x2): Conn_01x05, symbol Connector_Generic:Conn_01x05
- added R? (x4): 1k, Resistor_SMD:R_0805_2012Metric_Pad1.15x1.40mm_HandSolder, symbol Device:R
- added R?: 0, Resistor_SMD:R_0805_2012Metric_Pad1.15x1.40mm_HandSolder, symbol Device:R
- added R?: 10k, Resistor_SMD:R_0805_2012Metric_Pad1.15x1.40mm_HandSolder, symbol Device:R
- added R?: 330 k, Resistor_SMD:R_0805_2012Metric_Pad1.15x1.40mm_HandSolder, symbol Device:R
- added U? (x2): 6N137, Package_DIP:DIP-8_W7.62mm, symbol Isolator:6N137
Connections:
- net labels added: +3.3V, +3.3VP, +5V, +5VP, GND, GNDS, UARTMaster_Rx, UARTMaster_Tx, UARTSlave_RX, UARTSlave_TX
- wire segments 0 -> 68
Other:
- moved on the sheet: Q?

Commit message: Asignacion inicial de footprints
Parts:
- J401, J402: renamed from J?; footprint (none) -> Connector_PinHeader_2.54mm:PinHeader_1x05_P2.54mm_Vertical
- U401, U402: renamed from U?; symbol Isolator:6N137 -> ModPrincipal-rescue:6N137-Isolator
- gave numbers to parts that had none: 12

Commit message: Asignación de footprint y corrección de errores de ERC en esquematico
Parts:
- added TP401, TP402: TestPoint, TestPoint:TestPoint_Pad_D1.5mm, symbol Connector:TestPoint
Connections:
- net +3V3: now also C403.1
- net +5V: now also C404.1
- net UARTSlave_RX: now also TP402.1
- net UARTSlave_TX: now also TP401.1
Changed lines of the file:
@@
 EESchema Schematic File Version 4
-LIBS:ModPrincipal-cache
 EELAYER 30 0
 EELAYER END
@@
 Wire Wire Line
 	7300 2450 7150 2450
-Text HLabel 7300 2650 2    50   Input ~ 0
+Text HLabel 7800 2650 2    50   Input ~ 0
 UARTSlave_TX
-Wire Wire Line
-	7300 2650 7150 2650
-Text HLabel 7800 3750 2    50   Output ~ 0
+Text HLabel 8350 3750 2    50   Output ~ 0
 UARTSlave_RX
-Wire Wire Line
-	7800 3750 7600 3750
-Connection ~ 7600 3750
 $Comp
 L Connector_Generic:Conn_01x05 J401
@@
 L power:+3.3VP #PWR0407
 U 1 1 5EDBAED1
-P 4050 3250
-F 0 "#PWR0407" H 4200 3200 50  0001 C CNN
-F 1 "+3.3VP" H 4070 3393 50  0000 C CNN
-F 2 "" H 4050 3250 50  0001 C CNN
-F 3 "" H 4050 3250 50  0001 C CNN
-	1    4050 3250
-	1    0    0    -1
-$EndComp
-Wire Wire Line
-	4050 3250 4050 3350
-Wire Wire Line
-	4050 3350 3800 3350
+P 4450 3150
+F 0 "#PWR0407" H 4600 3100 50  0001 C CNN
+F 1 "+3.3VP" H 4470 3293 50  0000 C CNN
+F 2 "" H 4450 3150 50  0001 C CNN
+F 3 "" H 4450 3150 50  0001 C CNN
+	1    4450 3150
+	1    0    0    -1
+$EndComp
 $Comp
 L power:+5VP #PWR0403
 U 1 1 5EDC0A46
-P 3950 4000
-F 0 "#PWR0403" H 3950 3850 50  0001 C CNN
-F 1 "+5VP" H 3965 4173 50  0000 C CNN
-F 2 "" H 3950 4000 50  0001 C CNN
-F 3 "" H 3950 4000 50  0001 C CNN
-	1    3950 4000
-	1    0    0    -1
-$EndComp
-Wire Wire Line
-	3950 4000 3800 4000
+P 3250 3900
+F 0 "#PWR0403" H 3250 3750 50  0001 C CNN
+F 1 "+5VP" H 3265 4073 50  0000 C CNN
+F 2 "" H 3250 3900 50  0001 C CNN
+F 3 "" H 3250 3900 50  0001 C CNN
+	1    3250 3900
+	1    0    0    -1
+$EndComp
 Wire Wire Line
 	3800 4000 3800 3750
@@
 L power:GNDS #PWR0409
 U 1 1 5EDC3914
-P 4200 3700
-F 0 "#PWR0409" H 4200 3450 50  0001 C CNN
-F 1 "GNDS" H 4205 3527 50  0000 C CNN
-F 2 "" H 4200 3700 50  0001 C CNN
-F 3 "" H 4200 3700 50  0001 C CNN
-	1    4200 3700
-	1    0    0    -1
-$EndComp
-Wire Wire Line
-	4200 3700 4200 3650
-Wire Wire Line
-	4200 3650 3800 3650
+P 4550 3700
+F 0 "#PWR0409" H 4550 3450 50  0001 C CNN
+F 1 "GNDS" H 4555 3527 50  0000 C CNN
+F 2 "" H 4550 3700 50  0001 C CNN
+F 3 "" H 4550 3700 50  0001 C CNN
+	1    4550 3700
+	1    0    0    -1
+$EndComp
 Wire Wire Line
 	3800 3550 5150 3550
@@
 Wire Wire Line
 	3800 5000 4050 5000
+$Comp
+L Connector:TestPoint TP?
+U 1 1 5ED42166
+P 7450 2600
+AR Path="/5ECD8445/5ED42166" Ref="TP?"  Part="1"
+AR Path="/5ED20EE2/5ED42166" Ref="TP401"  Part="1"
+F 0 "TP401" H 7508 2718 50  0000 L CNN
+F 1 "TestPoint" H 7508 2627 50  0000 L CNN
+F 2 "TestPoint:TestPoint_Pad_D1.5mm" H 7650 2600 50  0001 C CNN
+F 3 "~" H 7650 2600 50  0001 C CNN
+	1    7450 2600
+	1    0    0    -1
+$EndComp
+Wire Wire Line
+	7450 2600 7450 2650
+Wire Wire Line
+	7800 2650 7450 2650
+Connection ~ 7450 2650
+Wire Wire Line
+	7450 2650 7150 2650
+$Comp
+L Connector:TestPoint TP?
+U 1 1 5ED4BF23
+P 8050 3700
+AR Path="/5ECD8445/5ED4BF23" Ref="TP?"  Part="1"
+AR Path="/5ED20EE2/5ED4BF23" Ref="TP402"  Part="1"
+F 0 "TP402" H 8108 3818 50  0000 L CNN
+F 1 "TestPoint" H 8108 3727 50  0000 L CNN
+F 2 "TestPoint:TestPoint_Pad_D1.5mm" H 8250 3700 50  0001 C CNN
+F 3 "~" H 8250 3700 50  0001 C CNN
+	1    8050 3700
+	1    0    0    -1
+$EndComp
+Wire Wire Line
+	8050 3700 8050 3750
+Wire Wire Line
+	8350 3750 8050 3750
+Connection ~ 7600 3750
+Connection ~ 8050 3750
+Wire Wire Line
+	8050 3750 7600 3750
+Wire Wire Line
+	9250 4700 9250 4800
+Wire Wire Line
+	8650 4700 8650 4800
+Wire Wire Line
+	4450 3150 4450 3350
+Wire Wire Line
+	4450 3350 4150 3350
+Wire Wire Line
+	4550 3700 4550 3650
+Wire Wire Line
+	4550 3650 4200 3650
+Wire Wire Line
+	3250 3900 3250 4000
+Wire Wire Line
+	3250 4000 3500 4000
+$Comp
+L power:PWR_FLAG #FLG0103
+U 1 1 5EE2396B
+P 4150 3200
+F 0 "#FLG0103" H 4150 3275 50  0001 C CNN
+F 1 "PWR_FLAG" H 4150 3373 50  0000 C CNN
+F 2 "" H 4150 3200 50  0001 C CNN
+F 3 "~" H 4150 3200 50  0001 C CNN
+	1    4150 3200
+	1    0    0    -1
+$EndComp
+$Comp
+L power:PWR_FLAG #FLG0104
+U 1 1 5EE270AB
+P 4200 3750
+F 0 "#FLG0104" H 4200 3825 50  0001 C CNN
+F 1 "PWR_FLAG" H 4200 3923 50  0000 C CNN
+F 2 "" H 4200 3750 50  0001 C CNN
+F 3 "~" H 4200 3750 50  0001 C CNN
+	1    4200 3750
+	-1   0    0    1
+$EndComp
+$Comp
+L power:PWR_FLAG #FLG0105
+U 1 1 5EE2DF7D
+P 3500 4100
+F 0 "#FLG0105" H 3500 4175 50  0001 C CNN
+F 1 "PWR_FLAG" H 3500 4273 50  0000 C CNN
+F 2 "" H 3500 4100 50  0001 C CNN
+F 3 "~" H 3500 4100 50  0001 C CNN
+	1    3500 4100
+	-1   0    0    1
+$EndComp
+Wire Wire Line
+	3500 4100 3500 4000
+Connection ~ 3500 4000
+Wire Wire Line
+	3500 4000 3800 4000
+Wire Wire Line
+	4200 3750 4200 3650
+Connection ~ 4200 3650
+Wire Wire Line
+	4200 3650 3800 3650
+Wire Wire Line
+	4150 3200 4150 3350
+Connection ~ 4150 3350
+Wire Wire Line
+	4150 3350 3800 3350
 $EndSCHEMATC

Commit message: Avance en trazado de pista Modulo principal
Connections:
- net +3V3: no longer R406.1, R407.1
- new net +3.3VA: R406.1, R407.1
Changed lines of the file:
@@
 	7250 3550 7250 3650
-$Comp
-L power:+3.3V #PWR0419
-U 1 1 5ED9F706
-P 7600 3250
-F 0 "#PWR0419" H 7600 3100 50  0001 C CNN
-F 1 "+3.3V" H 7615 3423 50  0000 C CNN
-F 2 "" H 7600 3250 50  0001 C CNN
-F 3 "" H 7600 3250 50  0001 C CNN
-	1    7600 3250
-	1    0    0    -1
-$EndComp
 $Comp
 L Device:R R?
@@
 Wire Wire Line
 	7250 3950 7150 3950
-$Comp
-L power:+3.3V #PWR0418
-U 1 1 5EDAF11A
-P 7300 1950
-F 0 "#PWR0418" H 7300 1800 50  0001 C CNN
-F 1 "+3.3V" H 7315 2123 50  0000 C CNN
-F 2 "" H 7300 1950 50  0001 C CNN
-F 3 "" H 7300 1950 50  0001 C CNN
-	1    7300 1950
-	1    0    0    -1
-$EndComp
 $Comp
 L Device:R R?
@@
 Wire Wire Line
 	4150 3350 3800 3350
+$Comp
+L power:+3.3VA #PWR?
+U 1 1 5EDA3AD4
+P 7300 1950
+AR Path="/5ED9C9D6/5EDA3AD4" Ref="#PWR?"  Part="1"
+AR Path="/5ED20EE2/5EDA3AD4" Ref="#PWR0101"  Part="1"
+F 0 "#PWR0101" H 7300 1800 50  0001 C CNN
+F 1 "+3.3VA" H 7315 2123 50  0000 C CNN
+F 2 "" H 7300 1950 50  0001 C CNN
+F 3 "" H 7300 1950 50  0001 C CNN
+	1    7300 1950
+	1    0    0    -1
+$EndComp
+$Comp
+L power:+3.3VA #PWR?
+U 1 1 5EDA70FC
+P 7600 3250
+AR Path="/5ED9C9D6/5EDA70FC" Ref="#PWR?"  Part="1"
+AR Path="/5ED20EE2/5EDA70FC" Ref="#PWR0102"  Part="1"
+F 0 "#PWR0102" H 7600 3100 50  0001 C CNN
+F 1 "+3.3VA" H 7615 3423 50  0000 C CNN
+F 2 "" H 7600 3250 50  0001 C CNN
+F 3 "" H 7600 3250 50  0001 C CNN
+	1    7600 3250
+	1    0    0    -1
+$EndComp
 $EndSCHEMATC

Commit message: Trazado completo de PCB modulo principal V1.0
Parts:
- removed J401, J402: Conn_01x05, Connector_PinHeader_2.54mm:PinHeader_1x05_P2.54mm_Vertical, symbol Connector_Generic:Conn_01x05
- added J401: Conn_02x05_Odd_Even, Connector_PinHeader_2.54mm:PinHeader_2x05_P2.54mm_Vertical, symbol Connector_Generic:Conn_02x05_Odd_Even
Connections:
- net +3V3 is gone; now on net +3.3VA: C403.1
- net +3.3VP: now also J401.10 (Pin_10), J401.9 (Pin_9)
- net +5VP: now also J401.1 (Pin_1), J401.2 (Pin_2)
- net GNDS: now also J401.3 (Pin_3), J401.4 (Pin_4)
- net UARTMaster_Rx: now also J401.5 (Pin_5), J401.6 (Pin_6)
- net UARTMaster_Tx: now also J401.7 (Pin_7), J401.8 (Pin_8)
Changed lines of the file:
@@
 encoding utf-8
 Sheet 4 8
-Title ""
-Date ""
-Rev ""
-Comp ""
-Comment1 ""
+Title "Probado - Modulo Principal"
+Date "2020-05-31"
+Rev "1.0"
+Comp "CESE - FIUBA"
+Comment1 "Gonzalo Gontad"
 Comment2 ""
 Comment3 ""
@@
 UARTSlave_RX
 $Comp
-L Connector_Generic:Conn_01x05 J401
-U 1 1 5EDB4016
-P 3600 3550
-F 0 "J401" H 3518 3125 50  0000 C CNN
-F 1 "Conn_01x05" H 3518 3216 50  0000 C CNN
-F 2 "Connector_PinHeader_2.54mm:PinHeader_1x05_P2.54mm_Vertical" H 3600 3550 50  0001 C CNN
-F 3 "~" H 3600 3550 50  0001 C CNN
-	1    3600 3550
-	-1   0    0    1
-$EndComp
-$Comp
 L power:+3.3VP #PWR0407
 U 1 1 5EDBAED1
@@
 L power:+5VP #PWR0403
 U 1 1 5EDC0A46
-P 3250 3900
-F 0 "#PWR0403" H 3250 3750 50  0001 C CNN
-F 1 "+5VP" H 3265 4073 50  0000 C CNN
-F 2 "" H 3250 3900 50  0001 C CNN
-F 3 "" H 3250 3900 50  0001 C CNN
-	1    3250 3900
+P 3950 3900
+F 0 "#PWR0403" H 3950 3750 50  0001 C CNN
+F 1 "+5VP" H 3965 4073 50  0000 C CNN
+F 2 "" H 3950 3900 50  0001 C CNN
+F 3 "" H 3950 3900 50  0001 C CNN
+	1    3950 3900
 	1    0    0    -1
 $EndComp
@@
 	3400 2400 3400 2500
 $Comp
-L power:+3.3V #PWR0420
-U 1 1 5EE1AF7E
-P 8650 4700
-F 0 "#PWR0420" H 8650 4550 50  0001 C CNN
-F 1 "+3.3V" H 8665 4873 50  0000 C CNN
-F 2 "" H 8650 4700 50  0001 C CNN
-F 3 "" H 8650 4700 50  0001 C CNN
-	1    8650 4700
-	1    0    0    -1
-$EndComp
-$Comp
 L power:+5V #PWR0422
 U 1 1 5EE1E069
@@
 	9250 5300 9250 5400
 $Comp
-L Connector_Generic:Conn_01x05 J402
-U 1 1 5EE59D4F
-P 3600 5000
-F 0 "J402" H 3518 4575 50  0000 C CNN
-F 1 "Conn_01x05" H 3518 4666 50  0000 C CNN
-F 2 "Connector_PinHeader_2.54mm:PinHeader_1x05_P2.54mm_Vertical" H 3600 5000 50  0001 C CNN
-F 3 "~" H 3600 5000 50  0001 C CNN
-	1    3600 5000
-	-1   0    0    1
-$EndComp
-$Comp
 L power:+3.3VP #PWR0408
 U 1 1 5EE59D55
-P 4050 4700
-F 0 "#PWR0408" H 4200 4650 50  0001 C CNN
-F 1 "+3.3VP" H 4070 4843 50  0000 C CNN
-F 2 "" H 4050 4700 50  0001 C CNN
-F 3 "" H 4050 4700 50  0001 C CNN
-	1    4050 4700
-	1    0    0    -1
-$EndComp
-Wire Wire Line
-	4050 4700 4050 4800
-Wire Wire Line
-	4050 4800 3800 4800
-$Comp
-L power:+5VP #PWR0404
-U 1 1 5EE59D5D
-P 3950 5450
-F 0 "#PWR0404" H 3950 5300 50  0001 C CNN
-F 1 "+5VP" H 3965 5623 50  0000 C CNN
-F 2 "" H 3950 5450 50  0001 C CNN
-F 3 "" H 3950 5450 50  0001 C CNN
-	1    3950 5450
-	1    0    0    -1
-$EndComp
-Wire Wire Line
-	3950 5450 3800 5450
-Wire Wire Line
-	3800 5450 3800 5200
+P 3050 3250
+F 0 "#PWR0408" H 3200 3200 50  0001 C CNN
+F 1 "+3.3VP" H 3070 3393 50  0000 C CNN
+F 2 "" H 3050 3250 50  0001 C CNN
+F 3 "" H 3050 3250 50  0001 C CNN
+	1    3050 3250
+	-1   0    0    -1
+$EndComp
+Wire Wire Line
+	3050 3250 3050 3350
+Wire Wire Line
+	3050 3350 3300 3350
 $Comp
 L power:GNDS #PWR0410
 U 1 1 5EE59D65
-P 4200 5150
-F 0 "#PWR0410" H 4200 4900 50  0001 C CNN
-F 1 "GNDS" H 4205 4977 50  0000 C CNN
-F 2 "" H 4200 5150 50  0001 C CNN
-F 3 "" H 4200 5150 50  0001 C CNN
-	1    4200 5150
-	1    0    0    -1
-$EndComp
-Wire Wire Line
-	4200 5150 4200 5100
-Wire Wire Line
-	4200 5100 3800 5100
-Text Label 4050 4900 0    50   ~ 0
+P 2900 3700
+F 0 "#PWR0410" H 2900 3450 50  0001 C CNN
+F 1 "GNDS" H 2905 3527 50  0000 C CNN
+F 2 "" H 2900 3700 50  0001 C CNN
+F 3 "" H 2900 3700 50  0001 C CNN
+	1    2900 3700
+	-1   0    0    -1
+$EndComp
+Wire Wire Line
+	2900 3700 2900 3650
+Wire Wire Line
+	2900 3650 3300 3650
+Text Label 3050 3450 2    50   ~ 0
 UARTMaster_Tx
-Text Label 4050 5000 0    50   ~ 0
+Text Label 3050 3550 2    50   ~ 0
 UARTMaster_Rx
 Wire Wire Line
-	4050 4900 3800 4900
-Wire Wire Line
-	3800 5000 4050 5000
+	3050 3450 3300 3450
+Wire Wire Line
+	3300 3550 3050 3550
 $Comp
 L Connector:TestPoint TP?
@@
 Wire Wire Line
 	4550 3650 4200 3650
-Wire Wire Line
-	3250 3900 3250 4000
-Wire Wire Line
-	3250 4000 3500 4000
 $Comp
 L power:PWR_FLAG #FLG0103
@@
 Wire Wire Line
 	3500 4100 3500 4000
-Connection ~ 3500 4000
 Wire Wire Line
 	3500 4000 3800 4000
@@
 	1    0    0    -1
 $EndComp
+$Comp
+L power:+3.3VA #PWR?
+U 1 1 5EDC62F4
+P 8650 4700
+AR Path="/5ED9C9D6/5EDC62F4" Ref="#PWR?"  Part="1"
+AR Path="/5ED20EE2/5EDC62F4" Ref="#PWR0110"  Part="1"
+F 0 "#PWR0110" H 8650 4550 50  0001 C CNN
+F 1 "+3.3VA" H 8665 4873 50  0000 C CNN
+F 2 "" H 8650 4700 50  0001 C CNN
+F 3 "" H 8650 4700 50  0001 C CNN
+	1    8650 4700
+	1    0    0    -1
+$EndComp
+$Comp
+L Connector_Generic:Conn_02x05_Odd_Even J401
+U 1 1 5EDD89D0
+P 3600 3550
+F 0 "J401" H 3650 3967 50  0000 C CNN
+F 1 "Conn_02x05_Odd_Even" H 3650 3876 50  0000 C CNN
+F 2 "Connector_PinHeader_2.54mm:PinHeader_2x05_P2.54mm_Vertical" H 3600 3550 50  0001 C CNN
+F 3 "~" H 3600 3550 50  0001 C CNN
+	1    3600 3550
+	-1   0    0    1
+$EndComp
+Wire Wire Line
+	3300 3750 3300 4000
+Wire Wire Line
+	3300 4000 3500 4000
+Connection ~ 3500 4000
+Wire Wire Line
+	3950 3900 3950 4000
+Wire Wire Line
+	3950 4000 3800 4000
+Connection ~ 3800 4000
 $EndSCHEMATC
