File: Hard/ModPrincipal/AnalogOut.sch (KiCad schematic (older format))
At the start: 12 parts

Commit message: Agrego fuente de alimentación
Parts:
- added C?: 100nF, Capacitor_SMD:C_0805_2012Metric_Pad1.15x1.40mm_HandSolder, symbol pspice:C
- added C?: 1nF, Capacitor_SMD:C_0805_2012Metric_Pad1.15x1.40mm_HandSolder, symbol pspice:C
- added U?: MCP4725xxx-xCH, Package_TO_SOT_SMD:SOT-23-6, symbol Analog_DACs:MCP4725xxx-xCH
Connections:
- net labels added: +3.3V, GND, SCL, SDA
- net labels removed: DAC
- wire segments 47 -> 57
Other:
- note removed: "0-3.3V\n"
- moved on the sheet: C?, R?, U?A, U?B, U?C, U?D, U?E

Commit message: Asignacion inicial de footprints
Parts:
- U301: renamed from U?; footprint (none) -> Package_SO:SOIC-14_3.9x8.7mm_P1.27mm
- U302: renamed from U?; symbol Analog_DACs:MCP4725xxx-xCH -> ModPrincipal-rescue:MCP4725xxx-xCH-Analog_DACs
- gave numbers to parts that had none: 9

Commit message: Asignación de footprint y corrección de errores de ERC en esquematico
Parts:
- added R305, R306: 4.7k, Resistor_SMD:R_0805_2012Metric_Pad1.15x1.40mm_HandSolder, symbol Device:R
- added TP301: TestPoint, TestPoint:TestPoint_Pad_D1.5mm, symbol Connector:TestPoint
Connections:
- net +3V3: now also R305.1, R306.1
- net SCL: now also R305.2
- net SDA: now also R306.2
- net at U301.3 (+), U302.1 (VOUT): now also TP301.1
Changed lines of the file:
@@
 EESchema Schematic File Version 4
-LIBS:ModPrincipal-cache
 EELAYER 30 0
 EELAYER END
@@
 $EndComp
 Wire Wire Line
-	8200 2550 8200 2650
-Wire Wire Line
 	8600 2200 8600 2350
 Wire Wire Line
@@
 Wire Wire Line
 	3100 4800 3100 4950
-Wire Wire Line
-	3100 5550 3100 5650
 $Comp
 L power:GNDA #PWR?
@@
 Connection ~ 6800 2350
 Wire Wire Line
-	6850 1900 5200 1900
+	6850 1900 5950 1900
 Wire Wire Line
 	6800 2750 6800 2850
@@
 	4300 2000 4400 2000
 Wire Wire Line
-	3550 1800 4400 1800
-Wire Wire Line
-	3550 1900 4400 1900
+	3550 1800 3800 1800
+Wire Wire Line
+	3550 1900 4150 1900
 $Comp
 L power:+3.3V #PWR0303
@@
 Text HLabel 3550 1800 0    50   Input ~ 0
 SCL
+$Comp
+L Device:R R?
+U 1 1 5ED1578C
+P 4150 1350
+AR Path="/5EC7150D/5ED1578C" Ref="R?"  Part="1"
+AR Path="/5ECD8445/5ED1578C" Ref="R306"  Part="1"
+F 0 "R306" V 3943 1350 50  0000 C CNN
+F 1 "4.7k" V 4034 1350 50  0000 C CNN
+F 2 "Resistor_SMD:R_0805_2012Metric_Pad1.15x1.40mm_HandSolder" V 4080 1350 50  0001 C CNN
+F 3 "~" H 4150 1350 50  0001 C CNN
+	1    4150 1350
+	1    0    0    -1
+$EndComp
+$Comp
+L Device:R R?
+U 1 1 5ED15792
+P 3800 1350
+AR Path="/5EC7150D/5ED15792" Ref="R?"  Part="1"
+AR Path="/5ECD8445/5ED15792" Ref="R305"  Part="1"
+F 0 "R305" V 3593 1350 50  0000 C CNN
+F 1 "4.7k" V 3684 1350 50  0000 C CNN
+F 2 "Resistor_SMD:R_0805_2012Metric_Pad1.15x1.40mm_HandSolder" V 3730 1350 50  0001 C CNN
+F 3 "~" H 3800 1350 50  0001 C CNN
+	1    3800 1350
+	1    0    0    -1
+$EndComp
+$Comp
+L power:+3.3V #PWR0317
+U 1 1 5ED18E3E
+P 3800 1050
+F 0 "#PWR0317" H 3800 900 50  0001 C CNN
+F 1 "+3.3V" H 3815 1223 50  0000 C CNN
+F 2 "" H 3800 1050 50  0001 C CNN
+F 3 "" H 3800 1050 50  0001 C CNN
+	1    3800 1050
+	1    0    0    -1
+$EndComp
+Wire Wire Line
+	3800 1050 3800 1200
+$Comp
+L power:+3.3V #PWR0318
+U 1 1 5ED1A1DA
+P 4150 1050
+F 0 "#PWR0318" H 4150 900 50  0001 C CNN
+F 1 "+3.3V" H 4165 1223 50  0000 C CNN
+F 2 "" H 4150 1050 50  0001 C CNN
+F 3 "" H 4150 1050 50  0001 C CNN
+	1    4150 1050
+	1    0    0    -1
+$EndComp
+Wire Wire Line
+	4150 1050 4150 1200
+Wire Wire Line
+	3800 1500 3800 1800
+Connection ~ 3800 1800
+Wire Wire Line
+	3800 1800 4400 1800
+Wire Wire Line
+	4150 1500 4150 1900
+Connection ~ 4150 1900
+Wire Wire Line
+	4150 1900 4400 1900
+$Comp
+L Connector:TestPoint TP301
+U 1 1 5ED26346
+P 5950 1850
+F 0 "TP301" H 6008 1968 50  0000 L CNN
+F 1 "TestPoint" H 6008 1877 50  0000 L CNN
+F 2 "TestPoint:TestPoint_Pad_D1.5mm" H 6150 1850 50  0001 C CNN
+F 3 "~" H 6150 1850 50  0001 C CNN
+	1    5950 1850
+	1    0    0    -1
+$EndComp
+Wire Wire Line
+	5950 1850 5950 1900
+Connection ~ 5950 1900
+Wire Wire Line
+	5950 1900 5200 1900
+Wire Wire Line
+	8200 2550 8200 2650
+Wire Wire Line
+	3100 5550 3100 5650
 $EndSCHEMATC

Commit message: Avance en trazado de pista Modulo principal
Connections:
- net +3V3 renamed +3.3VA
Changed lines of the file:
@@
-$EndComp
-$Comp
-L power:+3.3V #PWR0310
-U 1 1 5EDE3863
-P 4800 1450
-F 0 "#PWR0310" H 4800 1300 50  0001 C CNN
-F 1 "+3.3V" H 4815 1623 50  0000 C CNN
-F 2 "" H 4800 1450 50  0001 C CNN
-F 3 "" H 4800 1450 50  0001 C CNN
-	1    4800 1450
-	1    0    0    -1
 $EndComp
 $Comp
@@
 Wire Wire Line
 	3550 1900 4150 1900
-$Comp
-L power:+3.3V #PWR0303
-U 1 1 5EE3FB8C
-P 2150 1500
-F 0 "#PWR0303" H 2150 1350 50  0001 C CNN
-F 1 "+3.3V" H 2165 1673 50  0000 C CNN
-F 2 "" H 2150 1500 50  0001 C CNN
-F 3 "" H 2150 1500 50  0001 C CNN
-	1    2150 1500
-	1    0    0    -1
-$EndComp
 $Comp
 L power:GND #PWR0306
@@
 $EndComp
 $Comp
-L power:+3.3V #PWR0305
-U 1 1 5EE47B5D
-P 2600 1500
-F 0 "#PWR0305" H 2600 1350 50  0001 C CNN
-F 1 "+3.3V" H 2615 1673 50  0000 C CNN
-F 2 "" H 2600 1500 50  0001 C CNN
-F 3 "" H 2600 1500 50  0001 C CNN
-	1    2600 1500
-	1    0    0    -1
-$EndComp
-$Comp
 L power:GND #PWR0304
 U 1 1 5EE4B0A1
@@
 	1    0    0    -1
 $EndComp
-$Comp
-L power:+3.3V #PWR0317
-U 1 1 5ED18E3E
-P 3800 1050
-F 0 "#PWR0317" H 3800 900 50  0001 C CNN
-F 1 "+3.3V" H 3815 1223 50  0000 C CNN
-F 2 "" H 3800 1050 50  0001 C CNN
-F 3 "" H 3800 1050 50  0001 C CNN
-	1    3800 1050
-	1    0    0    -1
-$EndComp
 Wire Wire Line
 	3800 1050 3800 1200
-$Comp
-L power:+3.3V #PWR0318
-U 1 1 5ED1A1DA
-P 4150 1050
-F 0 "#PWR0318" H 4150 900 50  0001 C CNN
-F 1 "+3.3V" H 4165 1223 50  0000 C CNN
-F 2 "" H 4150 1050 50  0001 C CNN
-F 3 "" H 4150 1050 50  0001 C CNN
-	1    4150 1050
-	1    0    0    -1
-$EndComp
 Wire Wire Line
 	4150 1050 4150 1200
@@
 Wire Wire Line
 	3100 5550 3100 5650
+$Comp
+L power:+3.3VA #PWR?
+U 1 1 5EDC216A
+P 2150 1500
+AR Path="/5ED9C9D6/5EDC216A" Ref="#PWR?"  Part="1"
+AR Path="/5ECD8445/5EDC216A" Ref="#PWR0104"  Part="1"
+F 0 "#PWR0104" H 2150 1350 50  0001 C CNN
+F 1 "+3.3VA" H 2165 1673 50  0000 C CNN
+F 2 "" H 2150 1500 50  0001 C CNN
+F 3 "" H 2150 1500 50  0001 C CNN
+	1    2150 1500
+	1    0    0    -1
+$EndComp
+$Comp
+L power:+3.3VA #PWR?
+U 1 1 5EDD0A68
+P 2600 1500
+AR Path="/5ED9C9D6/5EDD0A68" Ref="#PWR?"  Part="1"
+AR Path="/5ECD8445/5EDD0A68" Ref="#PWR0105"  Part="1"
+F 0 "#PWR0105" H 2600 1350 50  0001 C CNN
+F 1 "+3.3VA" H 2615 1673 50  0000 C CNN
+F 2 "" H 2600 1500 50  0001 C CNN
+F 3 "" H 2600 1500 50  0001 C CNN
+	1    2600 1500
+	1    0    0    -1
+$EndComp
+$Comp
+L power:+3.3VA #PWR?
+U 1 1 5EDD9CD2
+P 3800 1050
+AR Path="/5ED9C9D6/5EDD9CD2" Ref="#PWR?"  Part="1"
+AR Path="/5ECD8445/5EDD9CD2" Ref="#PWR0106"  Part="1"
+F 0 "#PWR0106" H 3800 900 50  0001 C CNN
+F 1 "+3.3VA" H 3815 1223 50  0000 C CNN
+F 2 "" H 3800 1050 50  0001 C CNN
+F 3 "" H 3800 1050 50  0001 C CNN
+	1    3800 1050
+	1    0    0    -1
+$EndComp
+$Comp
+L power:+3.3VA #PWR?
+U 1 1 5EDDB311
+P 4150 1050
+AR Path="/5ED9C9D6/5EDDB311" Ref="#PWR?"  Part="1"
+AR Path="/5ECD8445/5EDDB311" Ref="#PWR0107"  Part="1"
+F 0 "#PWR0107" H 4150 900 50  0001 C CNN
+F 1 "+3.3VA" H 4165 1223 50  0000 C CNN
+F 2 "" H 4150 1050 50  0001 C CNN
+F 3 "" H 4150 1050 50  0001 C CNN
+	1    4150 1050
+	1    0    0    -1
+$EndComp
+$Comp
+L power:+3.3VA #PWR?
+U 1 1 5EDE1CF9
+P 4800 1450
+AR Path="/5ED9C9D6/5EDE1CF9" Ref="#PWR?"  Part="1"
+AR Path="/5ECD8445/5EDE1CF9" Ref="#PWR0108"  Part="1"
+F 0 "#PWR0108" H 4800 1300 50  0001 C CNN
+F 1 "+3.3VA" H 4815 1623 50  0000 C CNN
+F 2 "" H 4800 1450 50  0001 C CNN
+F 3 "" H 4800 1450 50  0001 C CNN
+	1    4800 1450
+	1    0    0    -1
+$EndComp
 $EndSCHEMATC
