File: Hard/ModPrincipal/CPU.sch (KiCad schematic (older format))
At the start: 6 parts

Commit message: Asignacion inicial de footprints
Parts:
- J801: renamed from J?; footprint (none) -> Connector_PinHeader_2.54mm:PinHeader_1x06_P2.54mm_Vertical
- R801, R802, R803, R804: renamed from R?; footprint (none) -> Resistor_SMD:R_0805_2012Metric_Pad1.15x1.40mm_HandSolder
- U801: renamed from U?; footprint (none) -> BluePill:BLUEPILL
Changed lines of the file:
@@
 EESchema Schematic File Version 4
+LIBS:ModPrincipal-cache
 EELAYER 30 0
 EELAYER END
 $Descr A4 11693 8268
 encoding utf-8
-Sheet 7 8
+Sheet 8 8
 Title ""
 Date ""
@@
 $EndDescr
 $Comp
-L BluePill:BP U?
+L BluePill:BP U801
 U 1 1 5ED9CBD1
 P 4650 3450
-F 0 "U?" H 4650 4703 60  0000 C CNN
+F 0 "U801" H 4650 4703 60  0000 C CNN
 F 1 "BP" H 4650 4597 60  0000 C CNN
-F 2 "" H 4550 4200 60  0001 C CNN
+F 2 "BluePill:BLUEPILL" H 4550 4200 60  0001 C CNN
 F 3 "" H 4550 4200 60  0001 C CNN
 	1    4650 3450
@@
 $EndComp
 $Comp
-L power:+5V #PWR?
+L power:+5V #PWR0803
 U 1 1 5ED9E304
 P 4800 2300
-F 0 "#PWR?" H 4800 2150 50  0001 C CNN
+F 0 "#PWR0803" H 4800 2150 50  0001 C CNN
 F 1 "+5V" H 4815 2473 50  0000 C CNN
 F 2 "" H 4800 2300 50  0001 C CNN
@@
 	4800 2300 4800 2400
 $Comp
-L power:GND #PWR?
+L power:GND #PWR0804
 U 1 1 5ED9EF1C
 P 4800 4600
-F 0 "#PWR?" H 4800 4350 50  0001 C CNN
+F 0 "#PWR0804" H 4800 4350 50  0001 C CNN
 F 1 "GND" H 4805 4427 50  0000 C CNN
 F 2 "" H 4800 4600 50  0001 C CNN
@@
 	5400 3750 5750 3750
 $Comp
-L power:GND #PWR?
+L power:GND #PWR0805
 U 1 1 5EDA9158
 P 5800 4750
-F 0 "#PWR?" H 5800 4500 50  0001 C CNN
+F 0 "#PWR0805" H 5800 4500 50  0001 C CNN
 F 1 "GND" H 5805 4577 50  0000 C CNN
 F 2 "" H 5800 4750 50  0001 C CNN
@@
 $EndComp
 $Comp
-L Device:R R?
+L Device:R R801
 U 1 1 5EDAA787
 P 5550 4450
-F 0 "R?" H 5620 4496 50  0000 L CNN
+F 0 "R801" H 5620 4496 50  0000 L CNN
 F 1 "R" H 5620 4405 50  0000 L CNN
-F 2 "" V 5480 4450 50  0001 C CNN
+F 2 "Resistor_SMD:R_0805_2012Metric_Pad1.15x1.40mm_HandSolder" V 5480 4450 50  0001 C CNN
 F 3 "~" H 5550 4450 50  0001 C CNN
 	1    5550 4450
@@
 $EndComp
 $Comp
-L Device:R R?
+L Device:R R802
 U 1 1 5EDAD0E8
 P 5800 4450
-F 0 "R?" H 5870 4496 50  0000 L CNN
+F 0 "R802" H 5870 4496 50  0000 L CNN
 F 1 "R" H 5870 4405 50  0000 L CNN
-F 2 "" V 5730 4450 50  0001 C CNN
+F 2 "Resistor_SMD:R_0805_2012Metric_Pad1.15x1.40mm_HandSolder" V 5730 4450 50  0001 C CNN
 F 3 "~" H 5800 4450 50  0001 C CNN
 	1    5800 4450
@@
 $EndComp
 $Comp
-L Device:R R?
+L Device:R R803
 U 1 1 5EDAD1E4
 P 6050 4450
-F 0 "R?" H 6120 4496 50  0000 L CNN
+F 0 "R803" H 6120 4496 50  0000 L CNN
 F 1 "R" H 6120 4405 50  0000 L CNN
-F 2 "" V 5980 4450 50  0001 C CNN
+F 2 "Resistor_SMD:R_0805_2012Metric_Pad1.15x1.40mm_HandSolder" V 5980 4450 50  0001 C CNN
 F 3 "~" H 6050 4450 50  0001 C CNN
 	1    6050 4450
@@
 $EndComp
 $Comp
-L Device:R R?
+L Device:R R804
 U 1 1 5EDAEC6A
 P 6300 4450
-F 0 "R?" H 6370 4496 50  0000 L CNN
+F 0 "R804" H 6370 4496 50  0000 L CNN
 F 1 "R" H 6370 4405 50  0000 L CNN
-F 2 "" V 6230 4450 50  0001 C CNN
+F 2 "Resistor_SMD:R_0805_2012Metric_Pad1.15x1.40mm_HandSolder" V 6230 4450 50  0001 C CNN
 F 3 "~" H 6300 4450 50  0001 C CNN
 	1    6300 4450
@@
 	5750 2850 5400 2850
 $Comp
-L Connector_Generic:Conn_01x06 J?
+L Connector_Generic:Conn_01x06 J801
 U 1 1 5EDBAA35
 P 2350 3750
-F 0 "J?" H 2268 3225 50  0000 C CNN
+F 0 "J801" H 2268 3225 50  0000 C CNN
 F 1 "Conn_01x06" H 2268 3316 50  0000 C CNN
-F 2 "" H 2350 3750 50  0001 C CNN
+F 2 "Connector_PinHeader_2.54mm:PinHeader_1x06_P2.54mm_Vertical" H 2350 3750 50  0001 C CNN
 F 3 "~" H 2350 3750 50  0001 C CNN
 	1    2350 3750
@@
 	3900 3850 2550 3850
 $Comp
-L power:+3.3V #PWR?
+L power:+3.3V #PWR0801
 U 1 1 5EDC0299
 P 2700 3250
-F 0 "#PWR?" H 2700 3100 50  0001 C CNN
+F 0 "#PWR0801" H 2700 3100 50  0001 C CNN
 F 1 "+3.3V" H 2715 3423 50  0000 C CNN
 F 2 "" H 2700 3250 50  0001 C CNN
@@
 	2700 3450 2550 3450
 $Comp
-L power:GND #PWR?
+L power:GND #PWR0802
 U 1 1 5EDC14E8
 P 2700 4100
-F 0 "#PWR?" H 2700 3850 50  0001 C CNN
+F 0 "#PWR0802" H 2700 3850 50  0001 C CNN
 F 1 "GND" H 2705 3927 50  0000 C CNN
 F 2 "" H 2700 4100 50  0001 C CNN

Commit message: Asignación de footprint y corrección de errores de ERC en esquematico
Parts:
- added TP801, TP802: TestPoint, TestPoint:TestPoint_Pad_D1.5mm, symbol Connector:TestPoint
Connections:
- wire segments 39 -> 43
- no-connect marks 0 -> 16
Changed lines of the file:
@@
 EESchema Schematic File Version 4
-LIBS:ModPrincipal-cache
 EELAYER 30 0
 EELAYER END
@@
 Wire Wire Line
 	5750 3250 5400 3250
-Text HLabel 5750 2950 2    50   Output ~ 0
+Text HLabel 6300 2950 2    50   Output ~ 0
 SCL
-Wire Wire Line
-	5750 2950 5400 2950
-Text HLabel 5750 2850 2    50   BiDi ~ 0
+Text HLabel 6300 2850 2    50   BiDi ~ 0
 SDA
-Wire Wire Line
-	5750 2850 5400 2850
 $Comp
 L Connector_Generic:Conn_01x06 J801
@@
 Wire Wire Line
 	2700 3950 2550 3950
+$Comp
+L Connector:TestPoint TP?
+U 1 1 5ED3083E
+P 5600 2650
+AR Path="/5ECD8445/5ED3083E" Ref="TP?"  Part="1"
+AR Path="/5ED9C9D6/5ED3083E" Ref="TP801"  Part="1"
+F 0 "TP801" H 5658 2768 50  0000 L CNN
+F 1 "TestPoint" H 5658 2677 50  0000 L CNN
+F 2 "TestPoint:TestPoint_Pad_D1.5mm" H 5800 2650 50  0001 C CNN
+F 3 "~" H 5800 2650 50  0001 C CNN
+	1    5600 2650
+	1    0    0    -1
+$EndComp
+$Comp
+L Connector:TestPoint TP?
+U 1 1 5ED31409
+P 6050 2650
+AR Path="/5ECD8445/5ED31409" Ref="TP?"  Part="1"
+AR Path="/5ED9C9D6/5ED31409" Ref="TP802"  Part="1"
+F 0 "TP802" H 6108 2768 50  0000 L CNN
+F 1 "TestPoint" H 6108 2677 50  0000 L CNN
+F 2 "TestPoint:TestPoint_Pad_D1.5mm" H 6250 2650 50  0001 C CNN
+F 3 "~" H 6250 2650 50  0001 C CNN
+	1    6050 2650
+	1    0    0    -1
+$EndComp
+Wire Wire Line
+	6300 2850 6050 2850
+Wire Wire Line
+	5400 2950 5600 2950
+Wire Wire Line
+	6050 2650 6050 2850
+Connection ~ 6050 2850
+Wire Wire Line
+	6050 2850 5400 2850
+Wire Wire Line
+	5600 2650 5600 2950
+Connection ~ 5600 2950
+Wire Wire Line
+	5600 2950 6300 2950
+NoConn ~ 3900 2650
+NoConn ~ 3900 2750
+NoConn ~ 3900 2850
+NoConn ~ 5400 2650
+NoConn ~ 5400 2750
+NoConn ~ 5400 3350
+NoConn ~ 5400 3450
+NoConn ~ 5400 3550
+NoConn ~ 5400 3850
+NoConn ~ 4500 2400
+NoConn ~ 4650 2400
+NoConn ~ 3900 3950
+NoConn ~ 3900 4050
+NoConn ~ 4500 4500
+NoConn ~ 4600 4500
+NoConn ~ 3900 4250
 $EndSCHEMATC

Commit message: Avance en place de componentes
Parts:
- removed U801: BP, BluePill:BLUEPILL, symbol BluePill:BP
- added R805, R806, R807, R808: R, Resistor_SMD:R_0805_2012Metric_Pad1.15x1.40mm_HandSolder, symbol Device:R
- added U801: BP2, BluePill:BLUEPILL2, symbol BluePill:BP2
Connections:
- wire segments 43 -> 55
- no-connect marks 16 -> 14
Other:
- moved on the sheet: R801, R802, R803, R804
Changed lines of the file:
@@
 EESchema Schematic File Version 4
-LIBS:ModPrincipal-cache
 EELAYER 30 0
 EELAYER END
@@
 $EndDescr
 $Comp
-L BluePill:BP U801
-U 1 1 5ED9CBD1
-P 4650 3450
-F 0 "U801" H 4650 4703 60  0000 C CNN
-F 1 "BP" H 4650 4597 60  0000 C CNN
-F 2 "BluePill:BLUEPILL" H 4550 4200 60  0001 C CNN
-F 3 "" H 4550 4200 60  0001 C CNN
-	1    4650 3450
-	1    0    0    -1
-$EndComp
-$Comp
 L power:+5V #PWR0803
 U 1 1 5ED9E304
@@
 L power:GND #PWR0805
 U 1 1 5EDA9158
-P 5800 4750
-F 0 "#PWR0805" H 5800 4500 50  0001 C CNN
-F 1 "GND" H 5805 4577 50  0000 C CNN
-F 2 "" H 5800 4750 50  0001 C CNN
-F 3 "" H 5800 4750 50  0001 C CNN
-	1    5800 4750
+P 6650 4750
+F 0 "#PWR0805" H 6650 4500 50  0001 C CNN
+F 1 "GND" H 6655 4577 50  0000 C CNN
+F 2 "" H 6650 4750 50  0001 C CNN
+F 3 "" H 6650 4750 50  0001 C CNN
+	1    6650 4750
 	1    0    0    -1
 $EndComp
@@
 L Device:R R801
 U 1 1 5EDAA787
-P 5550 4450
-F 0 "R801" H 5620 4496 50  0000 L CNN
-F 1 "R" H 5620 4405 50  0000 L CNN
-F 2 "Resistor_SMD:R_0805_2012Metric_Pad1.15x1.40mm_HandSolder" V 5480 4450 50  0001 C CNN
-F 3 "~" H 5550 4450 50  0001 C CNN
-	1    5550 4450
+P 6400 4450
+F 0 "R801" H 6470 4496 50  0000 L CNN
+F 1 "R" H 6470 4405 50  0000 L CNN
+F 2 "Resistor_SMD:R_0805_2012Metric_Pad1.15x1.40mm_HandSolder" V 6330 4450 50  0001 C CNN
+F 3 "~" H 6400 4450 50  0001 C CNN
+	1    6400 4450
 	1    0    0    -1
 $EndComp
@@
 L Device:R R802
 U 1 1 5EDAD0E8
-P 5800 4450
-F 0 "R802" H 5870 4496 50  0000 L CNN
-F 1 "R" H 5870 4405 50  0000 L CNN
-F 2 "Resistor_SMD:R_0805_2012Metric_Pad1.15x1.40mm_HandSolder" V 5730 4450 50  0001 C CNN
-F 3 "~" H 5800 4450 50  0001 C CNN
-	1    5800 4450
+P 6650 4450
+F 0 "R802" H 6720 4496 50  0000 L CNN
+F 1 "R" H 6720 4405 50  0000 L CNN
+F 2 "Resistor_SMD:R_0805_2012Metric_Pad1.15x1.40mm_HandSolder" V 6580 4450 50  0001 C CNN
+F 3 "~" H 6650 4450 50  0001 C CNN
+	1    6650 4450
 	1    0    0    -1
 $EndComp
@@
 L Device:R R803
 U 1 1 5EDAD1E4
-P 6050 4450
-F 0 "R803" H 6120 4496 50  0000 L CNN
-F 1 "R" H 6120 4405 50  0000 L CNN
-F 2 "Resistor_SMD:R_0805_2012Metric_Pad1.15x1.40mm_HandSolder" V 5980 4450 50  0001 C CNN
-F 3 "~" H 6050 4450 50  0001 C CNN
-	1    6050 4450
+P 6900 4450
+F 0 "R803" H 6970 4496 50  0000 L CNN
+F 1 "R" H 6970 4405 50  0000 L CNN
+F 2 "Resistor_SMD:R_0805_2012Metric_Pad1.15x1.40mm_HandSolder" V 6830 4450 50  0001 C CNN
+F 3 "~" H 6900 4450 50  0001 C CNN
+	1    6900 4450
 	1    0    0    -1
 $EndComp
@@
 L Device:R R804
 U 1 1 5EDAEC6A
-P 6300 4450
-F 0 "R804" H 6370 4496 50  0000 L CNN
-F 1 "R" H 6370 4405 50  0000 L CNN
-F 2 "Resistor_SMD:R_0805_2012Metric_Pad1.15x1.40mm_HandSolder" V 6230 4450 50  0001 C CNN
-F 3 "~" H 6300 4450 50  0001 C CNN
-	1    6300 4450
-	1    0    0    -1
-$EndComp
-Wire Wire Line
-	5400 4250 5550 4250
-Wire Wire Line
-	5550 4250 5550 4300
-Wire Wire Line
-	5400 4150 5800 4150
-Wire Wire Line
-	5800 4150 5800 4300
-Wire Wire Line
-	5400 4050 6050 4050
-Wire Wire Line
-	6050 4050 6050 4300
-Wire Wire Line
-	5400 3950 6300 3950
-Wire Wire Line
-	6300 3950 6300 4300
-Wire Wire Line
-	5550 4600 5550 4650
-Wire Wire Line
-	5550 4650 5800 4650
-Wire Wire Line
-	6300 4650 6300 4600
-Connection ~ 5800 4650
-Wire Wire Line
-	5800 4650 6050 4650
-Wire Wire Line
-	6050 4600 6050 4650
-Connection ~ 6050 4650
-Wire Wire Line
-	6050 4650 6300 4650
-Wire Wire Line
-	5800 4600 5800 4650
-Wire Wire Line
-	5800 4650 5800 4750
+P 7150 4450
+F 0 "R804" H 7220 4496 50  0000 L CNN
+F 1 "R" H 7220 4405 50  0000 L CNN
+F 2 "Resistor_SMD:R_0805_2012Metric_Pad1.15x1.40mm_HandSolder" V 7080 4450 50  0001 C CNN
+F 3 "~" H 7150 4450 50  0001 C CNN
+	1    7150 4450
+	1    0    0    -1
+$EndComp
+Wire Wire Line
+	6400 4600 6400 4650
+Wire Wire Line
+	6400 4650 6650 4650
+Wire Wire Line
+	7150 4650 7150 4600
+Connection ~ 6650 4650
+Wire Wire Line
+	6650 4650 6900 4650
+Wire Wire Line
+	6900 4600 6900 4650
+Connection ~ 6900 4650
+Wire Wire Line
+	6900 4650 7150 4650
+Wire Wire Line
+	6650 4600 6650 4650
+Wire Wire Line
+	6650 4650 6650 4750
 Text HLabel 3600 3150 0    50   Output ~ 0
 ModPowerOut
@@
 NoConn ~ 3900 3950
 NoConn ~ 3900 4050
-NoConn ~ 4500 4500
-NoConn ~ 4600 4500
 NoConn ~ 3900 4250
+$Comp
+L BluePill:BP2 U801
+U 1 1 5ED1A12B
+P 4650 3450
+F 0 "U801" H 4200 2500 60  0000 C CNN
+F 1 "BP2" H 4250 2400 60  0000 C CNN
+F 2 "BluePill:BLUEPILL2" H 4550 4200 60  0001 C CNN
+F 3 "" H 4550 4200 60  0001 C CNN
+	1    4650 3450
+	1    0    0    -1
+$EndComp
+$Comp
+L Device:R R805
+U 1 1 5EDB6A95
+P 6400 3700
+F 0 "R805" H 6470 3746 50  0000 L CNN
+F 1 "R" H 6470 3655 50  0000 L CNN
+F 2 "Resistor_SMD:R_0805_2012Metric_Pad1.15x1.40mm_HandSolder" V 6330 3700 50  0001 C CNN
+F 3 "~" H 6400 3700 50  0001 C CNN
+	1    6400 3700
+	1    0    0    -1
+$EndComp
+$Comp
+L Device:R R806
+U 1 1 5EDB6A9B
+P 6650 3700
+F 0 "R806" H 6720 3746 50  0000 L CNN
+F 1 "R" H 6720 3655 50  0000 L CNN
+F 2 "Resistor_SMD:R_0805_2012Metric_Pad1.15x1.40mm_HandSolder" V 6580 3700 50  0001 C CNN
+F 3 "~" H 6650 3700 50  0001 C CNN
+	1    6650 3700
+	1    0    0    -1
+$EndComp
+$Comp
+L Device:R R807
+U 1 1 5EDB6AA1
+P 6900 3700
+F 0 "R807" H 6970 3746 50  0000 L CNN
+F 1 "R" H 6970 3655 50  0000 L CNN
+F 2 "Resistor_SMD:R_0805_2012Metric_Pad1.15x1.40mm_HandSolder" V 6830 3700 50  0001 C CNN
+F 3 "~" H 6900 3700 50  0001 C CNN
+	1    6900 3700
+	1    0    0    -1
+$EndComp
+$Comp
+L Device:R R808
+U 1 1 5EDB6AA7
+P 7150 3700
+F 0 "R808" H 7220 3746 50  0000 L CNN
+F 1 "R" H 7220 3655 50  0000 L CNN
+F 2 "Resistor_SMD:R_0805_2012Metric_Pad1.15x1.40mm_HandSolder" V 7080 3700 50  0001 C CNN
+F 3 "~" H 7150 3700 50  0001 C CNN
+	1    7150 3700
+	1    0    0    -1
+$EndComp
+$Comp
+L power:+3.3V #PWR0806
+U 1 1 5EDB772B
+P 6650 3350
+F 0 "#PWR0806" H 6650 3200 50  0001 C CNN
+F 1 "+3.3V" H 6665 3523 50  0000 C CNN
+F 2 "" H 6650 3350 50  0001 C CNN
+F 3 "" H 6650 3350 50  0001 C CNN
+	1    6650 3350
+	1    0    0    -1
+$EndComp
+Wire Wire Line
+	6400 3550 6400 3450
+Wire Wire Line
+	6400 3450 6650 3450
+Wire Wire Line
+	7150 3450 7150 3550
+Wire Wire Line
+	6900 3550 6900 3450
+Connection ~ 6900 3450
+Wire Wire Line
+	6900 3450 7150 3450
+Wire Wire Line
+	6650 3550 6650 3450
+Connection ~ 6650 3450
+Wire Wire Line
+	6650 3450 6900 3450
+Wire Wire Line
+	6650 3350 6650 3450
+Wire Wire Line
+	7150 3850 7150 3950
+Wire Wire Line
+	6900 3850 6900 4050
+Wire Wire Line
+	6400 3850 6400 4250
+Wire Wire Line
+	5400 3950 7150 3950
+Connection ~ 7150 3950
+Wire Wire Line
+	7150 3950 7150 4300
+Wire Wire Line
+	5400 4050 6900 4050
+Connection ~ 6900 4050
+Wire Wire Line
+	6900 4050 6900 4300
+Wire Wire Line
+	5400 4150 6650 4150
+Wire Wire Line
+	6650 3850 6650 4150
+Connection ~ 6650 4150
+Wire Wire Line
+	6650 4150 6650 4300
+Wire Wire Line
+	5400 4250 6400 4250
+Connection ~ 6400 4250
+Wire Wire Line
+	6400 4250 6400 4300
 $EndSCHEMATC

Commit message: Avance en trazado de pista Modulo principal
Parts:
- added C801, C802: 100nF, Capacitor_SMD:C_0805_2012Metric_Pad1.15x1.40mm_HandSolder, symbol pspice:C
Connections:
- net +3V3 is gone; now on net +3.3VA: J801.6 (Pin_6), R805.1, R806.1, R807.1, R808.1
- net +5V: now also C801.1, C802.1
- net GND: now also C801.2, C802.2
- net ModIn0: now also U801.PB5; no longer U801.PB3
- net ModIn2: now also U801.PB3; no longer U801.PB5
- net ModOut0: now also U801.PA2; no longer U801.PA3
- net ModOut1: now also U801.PA3; no longer U801.PA4
- net ModOut2: now also U801.PA4; no longer U801.PA5
- net ModPowerOut: now also U801.PA5; no longer U801.PA2
- net +3.3VA: now reaches U801.3V3 (3.3V)
- no-connect marks 14 -> 13
Changed lines of the file:
@@
 Wire Wire Line
 	6650 4650 6650 4750
+Text HLabel 3600 3450 0    50   Output ~ 0
+ModPowerOut
 Text HLabel 3600 3150 0    50   Output ~ 0
-ModPowerOut
+ModOut0
 Text HLabel 3600 3250 0    50   Output ~ 0
-ModOut0
+ModOut1
 Text HLabel 3600 3350 0    50   Output ~ 0
-ModOut1
-Text HLabel 3600 3450 0    50   Output ~ 0
 ModOut2
 Wire Wire Line
@@
 Wire Wire Line
 	3600 3450 3900 3450
-Text HLabel 5750 3250 2    50   Input ~ 0
+Text HLabel 5750 3050 2    50   Input ~ 0
 ModIn0
 Text HLabel 5750 3150 2    50   Input ~ 0
 ModIn1
-Text HLabel 5750 3050 2    50   Input ~ 0
+Text HLabel 5750 3250 2    50   Input ~ 0
 ModIn2
 Wire Wire Line
@@
 Wire Wire Line
 	3900 3850 2550 3850
-$Comp
-L power:+3.3V #PWR0801
-U 1 1 5EDC0299
-P 2700 3250
-F 0 "#PWR0801" H 2700 3100 50  0001 C CNN
-F 1 "+3.3V" H 2715 3423 50  0000 C CNN
-F 2 "" H 2700 3250 50  0001 C CNN
-F 3 "" H 2700 3250 50  0001 C CNN
-	1    2700 3250
-	1    0    0    -1
-$EndComp
 Wire Wire Line
 	2700 3250 2700 3450
@@
 NoConn ~ 5400 3850
 NoConn ~ 4500 2400
-NoConn ~ 4650 2400
 NoConn ~ 3900 3950
 NoConn ~ 3900 4050
@@
 	1    0    0    -1
 $EndComp
-$Comp
-L power:+3.3V #PWR0806
-U 1 1 5EDB772B
+Wire Wire Line
+	6400 3550 6400 3450
+Wire Wire Line
+	6400 3450 6650 3450
+Wire Wire Line
+	7150 3450 7150 3550
+Wire Wire Line
+	6900 3550 6900 3450
+Connection ~ 6900 3450
+Wire Wire Line
+	6900 3450 7150 3450
+Wire Wire Line
+	6650 3550 6650 3450
+Connection ~ 6650 3450
+Wire Wire Line
+	6650 3450 6900 3450
+Wire Wire Line
+	6650 3350 6650 3450
+Wire Wire Line
+	7150 3850 7150 3950
+Wire Wire Line
+	6900 3850 6900 4050
+Wire Wire Line
+	6400 3850 6400 4250
+Wire Wire Line
+	5400 3950 7150 3950
+Connection ~ 7150 3950
+Wire Wire Line
+	7150 3950 7150 4300
+Wire Wire Line
+	5400 4050 6900 4050
+Connection ~ 6900 4050
+Wire Wire Line
+	6900 4050 6900 4300
+Wire Wire Line
+	5400 4150 6650 4150
+Wire Wire Line
+	6650 3850 6650 4150
+Connection ~ 6650 4150
+Wire Wire Line
+	6650 4150 6650 4300
+Wire Wire Line
+	5400 4250 6400 4250
+Connection ~ 6400 4250
+Wire Wire Line
+	6400 4250 6400 4300
+$Comp
+L power:+3.3VA #PWR0103
+U 1 1 5EDA1357
+P 4650 2400
+F 0 "#PWR0103" H 4650 2250 50  0001 C CNN
+F 1 "+3.3VA" H 4665 2573 50  0000 C CNN
+F 2 "" H 4650 2400 50  0001 C CNN
+F 3 "" H 4650 2400 50  0001 C CNN
+	1    4650 2400
+	1    0    0    -1
+$EndComp
+$Comp
+L power:+3.3VA #PWR0109
+U 1 1 5EDE7E13
 P 6650 3350
-F 0 "#PWR0806" H 6650 3200 50  0001 C CNN
-F 1 "+3.3V" H 6665 3523 50  0000 C CNN
+F 0 "#PWR0109" H 6650 3200 50  0001 C CNN
+F 1 "+3.3VA" H 6665 3523 50  0000 C CNN
 F 2 "" H 6650 3350 50  0001 C CNN
 F 3 "" H 6650 3350 50  0001 C CNN
@@
 	1    0    0    -1
 $EndComp
-Wire Wire Line
-	6400 3550 6400 3450
-Wire Wire Line
-	6400 3450 6650 3450
-Wire Wire Line
-	7150 3450 7150 3550
-Wire Wire Line
-	6900 3550 6900 3450
-Connection ~ 6900 3450
-Wire Wire Line
-	6900 3450 7150 3450
-Wire Wire Line
-	6650 3550 6650 3450
-Connection ~ 6650 3450
-Wire Wire Line
-	6650 3450 6900 3450
-Wire Wire Line
-	6650 3350 6650 3450
-Wire Wire Line
-	7150 3850 7150 3950
-Wire Wire Line
-	6900 3850 6900 4050
-Wire Wire Line
-	6400 3850 6400 4250
-Wire Wire Line
-	5400 3950 7150 3950
-Connection ~ 7150 3950
-Wire Wire Line
-	7150 3950 7150 4300
-Wire Wire Line
-	5400 4050 6900 4050
-Connection ~ 6900 4050
-Wire Wire Line
-	6900 4050 6900 4300
-Wire Wire Line
-	5400 4150 6650 4150
-Wire Wire Line
-	6650 3850 6650 4150
-Connection ~ 6650 4150
-Wire Wire Line
-	6650 4150 6650 4300
-Wire Wire Line
-	5400 4250 6400 4250
-Connection ~ 6400 4250
-Wire Wire Line
-	6400 4250 6400 4300
+$Comp
+L power:+3.3VA #PWR0110
+U 1 1 5EDEB176
+P 2700 3250
+F 0 "#PWR0110" H 2700 3100 50  0001 C CNN
+F 1 "+3.3VA" H 2715 3423 50  0000 C CNN
+F 2 "" H 2700 3250 50  0001 C CNN
+F 3 "" H 2700 3250 50  0001 C CNN
+	1    2700 3250
+	1    0    0    -1
+$EndComp
+$Comp
+L power:GND #PWR?
+U 1 1 5EE3F126
+P 2450 2250
+AR Path="/5ECD8445/5EE3F126" Ref="#PWR?"  Part="1"
+AR Path="/5ED9C9D6/5EE3F126" Ref="#PWR0808"  Part="1"
+F 0 "#PWR0808" H 2450 2000 50  0001 C CNN
+F 1 "GND" H 2455 2077 50  0000 C CNN
+F 2 "" H 2450 2250 50  0001 C CNN
+F 3 "" H 2450 2250 50  0001 C CNN
+	1    2450 2250
+	1    0    0    -1
+$EndComp
+$Comp
+L pspice:C C?
+U 1 1 5EE3F12C
+P 2450 1800
+AR Path="/5EC7150D/5EE3F12C" Ref="C?"  Part="1"
+AR Path="/5ECD8445/5EE3F12C" Ref="C?"  Part="1"
+AR Path="/5ED9C9D6/5EE3F12C" Ref="C802"  Part="1"
+F 0 "C802" H 2250 1650 50  0000 L CNN
+F 1 "100nF" H 2550 1650 50  0000 L CNN
+F 2 "Capacitor_SMD:C_0805_2012Metric_Pad1.15x1.40mm_HandSolder" H 2450 1800 50  0001 C CNN
+F 3 "~" H 2450 1800 50  0001 C CNN
+	1    2450 1800
+	1    0    0    -1
+$EndComp
+$Comp
+L pspice:C C?
+U 1 1 5EE3F132
+P 2000 1800
+AR Path="/5EC7150D/5EE3F132" Ref="C?"  Part="1"
+AR Path="/5ECD8445/5EE3F132" Ref="C?"  Part="1"
+AR Path="/5ED9C9D6/5EE3F132" Ref="C801"  Part="1"
+F 0 "C801" H 1800 1650 50  0000 L CNN
+F 1 "100nF" H 2100 1650 50  0000 L CNN
+F 2 "Capacitor_SMD:C_0805_2012Metric_Pad1.15x1.40mm_HandSolder" H 2000 1800 50  0001 C CNN
+F 3 "~" H 2000 1800 50  0001 C CNN
+	1    2000 1800
+	1    0    0    -1
+$EndComp
+$Comp
+L power:GND #PWR?
+U 1 1 5EE3F138
+P 2000 2250
+AR Path="/5ECD8445/5EE3F138" Ref="#PWR?"  Part="1"
+AR Path="/5ED9C9D6/5EE3F138" Ref="#PWR0806"  Part="1"
+F 0 "#PWR0806" H 2000 2000 50  0001 C CNN
+F 1 "GND" H 2005 2077 50  0000 C CNN
+F 2 "" H 2000 2250 50  0001 C CNN
+F 3 "" H 2000 2250 50  0001 C CNN
+	1    2000 2250
+	1    0    0    -1
+$EndComp
+Wire Wire Line
+	2000 2250 2000 2050
+Wire Wire Line
+	2450 2050 2450 2250
+Wire Wire Line
+	2450 1550 2450 1350
+Wire Wire Line
+	2000 1350 2000 1550
+$Comp
+L power:+5V #PWR0801
+U 1 1 5EE419C5
+P 2000 1350
+F 0 "#PWR0801" H 2000 1200 50  0001 C CNN
+F 1 "+5V" H 2015 1523 50  0000 C CNN
+F 2 "" H 2000 1350 50  0001 C CNN
+F 3 "" H 2000 1350 50  0001 C CNN
+	1    2000 1350
+	1    0    0    -1
+$EndComp
+$Comp
+L power:+5V #PWR0807
+U 1 1 5EE4C9B5
+P 2450 1350
+F 0 "#PWR0807" H 2450 1200 50  0001 C CNN
+F 1 "+5V" H 2465 1523 50  0000 C CNN
+F 2 "" H 2450 1350 50  0001 C CNN
+F 3 "" H 2450 1350 50  0001 C CNN
+	1    2450 1350
+	1    0    0    -1
+$EndComp
 $EndSCHEMATC

Commit message: Trazado completo de PCB modulo principal V1.0
Parts:
- removed J801: Conn_01x06, Connector_PinHeader_2.54mm:PinHeader_1x06_P2.54mm_Vertical, symbol Connector_Generic:Conn_01x06
Connections:
- net ModIn0: now also U801.PA5; no longer U801.PB5
- net ModIn1: now also U801.PA6; no longer U801.PB4
- net ModIn2: now also U801.PA7; no longer U801.PB3
- net ModPowerOut: now also U801.PB0; no longer U801.PA5
- no-connect marks 13 -> 17
Changed lines of the file:
@@
 encoding utf-8
 Sheet 8 8
-Title ""
-Date ""
-Rev ""
-Comp ""
-Comment1 ""
+Title "Probado - Modulo Principal"
+Date "2020-05-31"
+Rev "1.0"
+Comp "CESE - FIUBA"
+Comment1 "Gonzalo Gontad"
 Comment2 ""
 Comment3 ""
@@
 Wire Wire Line
 	6650 4650 6650 4750
-Text HLabel 3600 3450 0    50   Output ~ 0
+Text HLabel 3600 3750 0    50   Output ~ 0
 ModPowerOut
 Text HLabel 3600 3150 0    50   Output ~ 0
@@
 	3600 3350 3900 3350
 Wire Wire Line
-	3600 3450 3900 3450
-Text HLabel 5750 3050 2    50   Input ~ 0
+	3600 3750 3900 3750
+Text HLabel 3550 3450 0    50   Input ~ 0
 ModIn0
-Text HLabel 5750 3150 2    50   Input ~ 0
+Text HLabel 3550 3550 0    50   Input ~ 0
 ModIn1
-Text HLabel 5750 3250 2    50   Input ~ 0
+Text HLabel 3550 3650 0    50   Input ~ 0
 ModIn2
 Wire Wire Line
-	5750 3050 5400 3050
-Wire Wire Line
-	5400 3150 5750 3150
-Wire Wire Line
-	5750 3250 5400 3250
+	3550 3650 3900 3650
+Wire Wire Line
+	3900 3550 3550 3550
+Wire Wire Line
+	3550 3450 3900 3450
 Text HLabel 6300 2950 2    50   Output ~ 0
 SCL
 Text HLabel 6300 2850 2    50   BiDi ~ 0
 SDA
-$Comp
-L Connector_Generic:Conn_01x06 J801
-U 1 1 5EDBAA35
-P 2350 3750
-F 0 "J801" H 2268 3225 50  0000 C CNN
-F 1 "Conn_01x06" H 2268 3316 50  0000 C CNN
-F 2 "Connector_PinHeader_2.54mm:PinHeader_1x06_P2.54mm_Vertical" H 2350 3750 50  0001 C CNN
-F 3 "~" H 2350 3750 50  0001 C CNN
-	1    2350 3750
-	-1   0    0    1
-$EndComp
-Wire Wire Line
-	2550 3550 3900 3550
-Wire Wire Line
-	3900 3650 2550 3650
-Wire Wire Line
-	2550 3750 3900 3750
-Wire Wire Line
-	3900 3850 2550 3850
-Wire Wire Line
-	2700 3250 2700 3450
-Wire Wire Line
-	2700 3450 2550 3450
-$Comp
-L power:GND #PWR0802
-U 1 1 5EDC14E8
-P 2700 4100
-F 0 "#PWR0802" H 2700 3850 50  0001 C CNN
-F 1 "GND" H 2705 3927 50  0000 C CNN
-F 2 "" H 2700 4100 50  0001 C CNN
-F 3 "" H 2700 4100 50  0001 C CNN
-	1    2700 4100
-	1    0    0    -1
-$EndComp
-Wire Wire Line
-	2700 4100 2700 3950
-Wire Wire Line
-	2700 3950 2550 3950
 $Comp
 L Connector:TestPoint TP?
@@
 $EndComp
 $Comp
-L power:+3.3VA #PWR0110
-U 1 1 5EDEB176
-P 2700 3250
-F 0 "#PWR0110" H 2700 3100 50  0001 C CNN
-F 1 "+3.3VA" H 2715 3423 50  0000 C CNN
-F 2 "" H 2700 3250 50  0001 C CNN
-F 3 "" H 2700 3250 50  0001 C CNN
-	1    2700 3250
-	1    0    0    -1
-$EndComp
-$Comp
 L power:GND #PWR?
 U 1 1 5EE3F126
@@
 	1    0    0    -1
 $EndComp
+NoConn ~ 3900 3850
+NoConn ~ 5400 3250
+NoConn ~ 5400 3150
+NoConn ~ 5400 3050
 $EndSCHEMATC
