File: Hard/ModPrincipal/Fuente.sch (KiCad schematic (older format))
At the start: 16 parts

Commit message: Asignacion inicial de footprints
Parts:
- C501, C502, C504, C506, C507: renamed from C?; footprint (none) -> Capacitor_SMD:C_1206_3216Metric_Pad1.42x1.75mm_HandSolder
- C503: renamed from C?; footprint (none) -> Capacitor_THT:CP_Radial_D8.0mm_P3.50mm
- C505: renamed from C?; value CAP -> 100nF; footprint (none) -> Capacitor_SMD:C_0805_2012Metric_Pad1.15x1.40mm_HandSolder
- U503: renamed from U?; footprint (none) -> Package_TO_SOT_THT:TO-220-3_Vertical
- gave numbers to parts that had none: 8

Commit message: Asignación de footprint y corrección de errores de ERC en esquematico
Parts:
- removed F501: Fuse, symbol Device:Fuse
- removed J502: Conn_01x02, symbol Connector_Generic:Conn_01x02
- added R501, R502, R503: 1, Resistor_SMD:R_0805_2012Metric_Pad1.15x1.40mm_HandSolder, symbol Device:R
- added TP501, TP502, TP503: TestPoint, TestPoint:TestPoint_Pad_D1.5mm, symbol Connector:TestPoint
- D501: footprint Package_TO_SOT_SMD:TO-269AA -> Package_SO:SO-4_4.4x4.3mm_P2.54mm
- J501: footprint (none) -> TerminalBlock:TerminalBlock_bornier-3_P5.08mm
- J503: footprint (none) -> TerminalBlock:TerminalBlock_bornier-2_P5.08mm
Connections:
- net labels added: GNDA
- wire segments 59 -> 73
Other:
- note removed: "Salida 220v al transformador"

Commit message: Avance en trazado de pista Modulo principal
Parts:
- removed D502: 1N4007, Diode_THT:D_DO-41_SOD81_P10.16mm_Horizontal, symbol Diode:1N4007
Connections:
- net at J503.1 (Pin_1): now also D501.2 (~~); no longer D501.1 (~~)
- net at J503.2 (Pin_2): now also D501.1 (~~); no longer D501.2 (~~)
Changed lines of the file:
@@
 L Connector_Generic:Conn_01x02 J503
 U 1 1 5ED063FA
-P 6450 1950
-F 0 "J503" V 6530 1942 50  0000 L CNN
-F 1 "Conn_01x02" H 6530 1851 50  0000 L CNN
-F 2 "TerminalBlock:TerminalBlock_bornier-2_P5.08mm" H 6450 1950 50  0001 C CNN
-F 3 "~" H 6450 1950 50  0001 C CNN
-	1    6450 1950
-	-1   0    0    1
+P 6450 1850
+F 0 "J503" V 6530 1842 50  0000 L CNN
+F 1 "Conn_01x02" H 6530 1751 50  0000 L CNN
+F 2 "TerminalBlock:TerminalBlock_bornier-2_P5.08mm" H 6450 1850 50  0001 C CNN
+F 3 "~" H 6450 1850 50  0001 C CNN
+	1    6450 1850
+	-1   0    0    -1
 $EndComp
 $Comp
@@
 	1    0    0    -1
 $EndComp
-$Comp
-L Diode:1N4007 D502
-U 1 1 5ED28BF5
-P 10500 2150
-F 0 "D502" V 10454 2229 50  0000 L CNN
-F 1 "1N4007" V 10545 2229 50  0000 L CNN
-F 2 "Diode_THT:D_DO-41_SOD81_P10.16mm_Horizontal" H 10500 1975 50  0001 C CNN
-F 3 "http://www.vishay.com/docs/88503/1n4001.pdf" H 10500 2150 50  0001 C CNN
-	1    10500 2150
-	0    1    1    0
-$EndComp
-Wire Wire Line
-	10500 2000 10500 1950
-Wire Wire Line
-	10500 1950 10050 1950
-$Comp
-L power:GND #PWR0518
-U 1 1 5ED2ABE3
-P 10500 2350
-F 0 "#PWR0518" H 10500 2100 50  0001 C CNN
-F 1 "GND" H 10505 2177 50  0000 C CNN
-F 2 "" H 10500 2350 50  0001 C CNN
-F 3 "" H 10500 2350 50  0001 C CNN
-	1    10500 2350
-	1    0    0    -1
-$EndComp
-Wire Wire Line
-	10500 2300 10500 2350
 $Comp
 L power:+3.3V #PWR0514
@@
 	-1   0    0    1
 $EndComp
-Connection ~ 10500 1950
 Wire Wire Line
 	9800 1950 10050 1950
@@
 Wire Wire Line
 	10750 1900 10750 1950
-Wire Wire Line
-	10750 1950 10500 1950
 Wire Wire Line
 	2650 1500 2300 1500
@@
 Wire Wire Line
 	2450 1700 3000 1700
+Wire Wire Line
+	10050 1950 10750 1950
 $EndSCHEMATC

Commit message: Inicio placement de componentes en Modulos Adicionales
Parts:
- J501: footprint TerminalBlock:TerminalBlock_bornier-3_P5.08mm -> Conectores:TerminalBlock_bornier-3_P5.00mm
- J503: footprint TerminalBlock:TerminalBlock_bornier-2_P5.08mm -> Conectores:TerminalBlock_bornier-2_P5.00mm
Changed lines of the file:
@@
 EESchema Schematic File Version 4
-LIBS:ModPrincipal-cache
 EELAYER 30 0
 EELAYER END
@@
 F 0 "J501" H 2018 1275 50  0000 C CNN
 F 1 "Conn_01x03" H 2018 1366 50  0000 C CNN
-F 2 "TerminalBlock:TerminalBlock_bornier-3_P5.08mm" H 2100 1600 50  0001 C CNN
+F 2 "Conectores:TerminalBlock_bornier-3_P5.00mm" H 2100 1600 50  0001 C CNN
 F 3 "~" H 2100 1600 50  0001 C CNN
 	1    2100 1600
@@
 F 0 "J503" V 6530 1842 50  0000 L CNN
 F 1 "Conn_01x02" H 6530 1751 50  0000 L CNN
-F 2 "TerminalBlock:TerminalBlock_bornier-2_P5.08mm" H 6450 1850 50  0001 C CNN
+F 2 "Conectores:TerminalBlock_bornier-2_P5.00mm" H 6450 1850 50  0001 C CNN
 F 3 "~" H 6450 1850 50  0001 C CNN
 	1    6450 1850
