File: Hard/ModPrincipal/Puerto.sch (KiCad schematic (older format))
At the start: 2 parts

Commit message: Asignacion inicial de footprints
Parts:
- J601: renamed from J?; footprint (none) -> Connector_PinSocket_2.54mm:PinSocket_2x10_P2.54mm_Horizontal
- J602: renamed from J?; footprint (none) -> Connector_PinSocket_2.54mm:PinSocket_2x05_P2.54mm_Horizontal
Changed lines of the file:
@@
 EESchema Schematic File Version 4
+LIBS:ModPrincipal-cache
 EELAYER 30 0
 EELAYER END
 $Descr A4 11693 8268
 encoding utf-8
-Sheet 8 8
+Sheet 6 8
 Title ""
 Date ""
@@
 $EndDescr
 $Comp
-L Connector_Generic:Conn_02x05_Odd_Even J?
+L Connector_Generic:Conn_02x05_Odd_Even J602
 U 1 1 5EE5AF19
 P 3850 1800
-F 0 "J?" H 3900 2217 50  0000 C CNN
+F 0 "J602" H 3900 2217 50  0000 C CNN
 F 1 "Conn_02x05_Odd_Even" H 3900 2126 50  0000 C CNN
-F 2 "" H 3850 1800 50  0001 C CNN
+F 2 "Connector_PinSocket_2.54mm:PinSocket_2x05_P2.54mm_Horizontal" H 3850 1800 50  0001 C CNN
 F 3 "~" H 3850 1800 50  0001 C CNN
 	1    3850 1800
@@
 In_Analog1
 $Comp
-L power:GND #PWR?
+L power:GND #PWR0603
 U 1 1 5EE71424
 P 4200 3850
-F 0 "#PWR?" H 4200 3600 50  0001 C CNN
+F 0 "#PWR0603" H 4200 3600 50  0001 C CNN
 F 1 "GND" H 4205 3677 50  0000 C CNN
 F 2 "" H 4200 3850 50  0001 C CNN
@@
 $EndComp
 $Comp
-L power:GNDA #PWR?
+L power:GNDA #PWR0601
 U 1 1 5EE71C71
 P 2500 3150
-F 0 "#PWR?" H 2500 2900 50  0001 C CNN
+F 0 "#PWR0601" H 2500 2900 50  0001 C CNN
 F 1 "GNDA" H 2505 2977 50  0000 C CNN
 F 2 "" H 2500 3150 50  0001 C CNN
@@
 $EndComp
 $Comp
-L power:+12V #PWR?
+L power:+12V #PWR0604
 U 1 1 5EE72298
 P 4450 3250
-F 0 "#PWR?" H 4450 3100 50  0001 C CNN
+F 0 "#PWR0604" H 4450 3100 50  0001 C CNN
 F 1 "+12V" H 4465 3423 50  0000 C CNN
 F 2 "" H 4450 3250 50  0001 C CNN
@@
 $EndComp
 $Comp
-L power:+5V #PWR?
+L power:+5V #PWR0605
 U 1 1 5EE727FD
 P 4550 3450
-F 0 "#PWR?" H 4550 3300 50  0001 C CNN
+F 0 "#PWR0605" H 4550 3300 50  0001 C CNN
 F 1 "+5V" H 4565 3623 50  0000 C CNN
 F 2 "" H 4550 3450 50  0001 C CNN
@@
 $EndComp
 $Comp
-L power:+3.3V #PWR?
+L power:+3.3V #PWR0606
 U 1 1 5EE72A4A
 P 4700 3600
-F 0 "#PWR?" H 4700 3450 50  0001 C CNN
+F 0 "#PWR0606" H 4700 3450 50  0001 C CNN
 F 1 "+3.3V" H 4715 3773 50  0000 C CNN
 F 2 "" H 4700 3600 50  0001 C CNN
@@
 	3350 3300 3550 3300
 $Comp
-L Connector_Generic:Conn_02x10_Odd_Even J?
+L Connector_Generic:Conn_02x10_Odd_Even J601
 U 1 1 5EE8E115
 P 3750 3200
-F 0 "J?" H 3800 3817 50  0000 C CNN
+F 0 "J601" H 3800 3817 50  0000 C CNN
 F 1 "Conn_02x10_Odd_Even" H 3800 3726 50  0000 C CNN
-F 2 "" H 3750 3200 50  0001 C CNN
+F 2 "Connector_PinSocket_2.54mm:PinSocket_2x10_P2.54mm_Horizontal" H 3750 3200 50  0001 C CNN
 F 3 "~" H 3750 3200 50  0001 C CNN
 	1    3750 3200
@@
 Connection ~ 2500 3100
 $Comp
-L power:GNDA #PWR?
+L power:GNDA #PWR0607
 U 1 1 5EEABF2C
 P 4950 3050
-F 0 "#PWR?" H 4950 2800 50  0001 C CNN
+F 0 "#PWR0607" H 4950 2800 50  0001 C CNN
 F 1 "GNDA" H 4955 2877 50  0000 C CNN
 F 2 "" H 4950 3050 50  0001 C CNN
@@
 Connection ~ 4200 3000
 $Comp
-L power:GNDPWR #PWR?
+L power:GNDPWR #PWR0602
 U 1 1 5EEC9156
 P 3350 2100
-F 0 "#PWR?" H 3350 1900 50  0001 C CNN
+F 0 "#PWR0602" H 3350 1900 50  0001 C CNN
 F 1 "GNDPWR" H 3354 1946 50  0000 C CNN
 F 2 "" H 3350 2050 50  0001 C CNN

Commit message: Asignación de footprint y corrección de errores de ERC en esquematico
Connections:
- no-connect marks 0 -> 4
Changed lines of the file:
@@
 EESchema Schematic File Version 4
-LIBS:ModPrincipal-cache
 EELAYER 30 0
 EELAYER END
@@
 Text HLabel 3350 1800 0    50   Input ~ 0
 Out_N_220
+NoConn ~ 3650 1900
+NoConn ~ 4150 1900
+NoConn ~ 4150 1700
+NoConn ~ 3650 1700
 $EndSCHEMATC

Commit message: Avance en trazado de pista Modulo principal
Parts:
- J602: footprint Connector_PinSocket_2.54mm:PinSocket_2x05_P2.54mm_Horizontal -> Connector:PinSocket_2x03_Doble_Paso_P2.54mm_Horizontal
Changed lines of the file:
@@
 F 0 "J602" H 3900 2217 50  0000 C CNN
 F 1 "Conn_02x05_Odd_Even" H 3900 2126 50  0000 C CNN
-F 2 "Connector_PinSocket_2.54mm:PinSocket_2x05_P2.54mm_Horizontal" H 3850 1800 50  0001 C CNN
+F 2 "Connector:PinSocket_2x03_Doble_Paso_P2.54mm_Horizontal" H 3850 1800 50  0001 C CNN
 F 3 "~" H 3850 1800 50  0001 C CNN
 	1    3850 1800
