File: Hard/ModAdicionales/Mod_Temp_Driver/Mod_Temp_Driver.sch (KiCad schematic (older format))
At the start: 3 parts

Commit message: Inicio Modulos Adicionales
Parts:
- removed J?: Conn_02x10_Odd_Even, symbol Connector_Generic:Conn_02x10_Odd_Even
- removed J?: Conn_02x05_Odd_Even, symbol Connector_Generic:Conn_02x05_Odd_Even
- removed K?: G5LE-1, Relay_THT:Relay_SPDT_Omron-G5LE-1, symbol Relay:G5LE-1
Connections:
- no-connect marks 4 -> 0
Changed lines of the file:
@@
 EESchema Schematic File Version 4
+LIBS:Mod_Temp_Driver-cache
 EELAYER 30 0
 EELAYER END
 $Descr A4 11693 8268
 encoding utf-8
-Sheet 1 1
+Sheet 1 3
 Title ""
 Date ""
@@
 Comment4 ""
 $EndDescr
-$Comp
-L Connector_Generic:Conn_02x10_Odd_Even J?
-U 1 1 5EEA125B
-P 3950 4900
-F 0 "J?" H 4000 5517 50  0000 C CNN
-F 1 "Conn_02x10_Odd_Even" H 4000 5426 50  0000 C CNN
-F 2 "" H 3950 4900 50  0001 C CNN
-F 3 "~" H 3950 4900 50  0001 C CNN
-	1    3950 4900
-	1    0    0    -1
-$EndComp
-$Comp
-L Connector_Generic:Conn_02x05_Odd_Even J?
-U 1 1 5EEA1AD2
-P 3850 2650
-F 0 "J?" H 3900 3067 50  0000 C CNN
-F 1 "Conn_02x05_Odd_Even" H 3900 2976 50  0000 C CNN
-F 2 "" H 3850 2650 50  0001 C CNN
-F 3 "~" H 3850 2650 50  0001 C CNN
-	1    3850 2650
-	1    0    0    -1
-$EndComp
-Text Label 2950 2650 0    50   ~ 0
-In_N_220
-Text Label 2950 2450 0    50   ~ 0
-In_L_220
-$Comp
-L power:GNDPWR #PWR?
-U 1 1 5EEA36E3
-P 3400 2950
-F 0 "#PWR?" H 3400 2750 50  0001 C CNN
-F 1 "GNDPWR" H 3404 2796 50  0000 C CNN
-F 2 "" H 3400 2900 50  0001 C CNN
-F 3 "" H 3400 2900 50  0001 C CNN
-	1    3400 2950
-	1    0    0    -1
-$EndComp
-Wire Wire Line
-	3400 2950 3400 2850
-Wire Wire Line
-	3400 2850 3650 2850
-Wire Wire Line
-	3650 2850 4150 2850
-Connection ~ 3650 2850
-Wire Wire Line
-	4150 2650 3650 2650
-Wire Wire Line
-	3650 2650 2950 2650
-Connection ~ 3650 2650
-Wire Wire Line
-	4150 2450 3650 2450
-Wire Wire Line
-	3650 2450 2950 2450
-Connection ~ 3650 2450
-Text Label 3100 4500 0    50   ~ 0
-Out_Analog0
-Text Label 3100 4700 0    50   ~ 0
-Out_Analog1
-Text Label 3100 4900 0    50   ~ 0
-In_Digital0
-Text Label 3100 5000 0    50   ~ 0
-In_Digital1
-Text Label 3100 5100 0    50   ~ 0
-In_Digital2
-Text Label 3100 5200 0    50   ~ 0
-Out_Digital0
-Text Label 3100 5300 0    50   ~ 0
-Out_Digital1
-Text Label 3100 5400 0    50   ~ 0
-Out_Digital2
-Text Label 4900 4600 2    50   ~ 0
-In_Analog0
-$Comp
-L power:+12V #PWR?
-U 1 1 5EEA8D36
-P 4650 4950
-F 0 "#PWR?" H 4650 4800 50  0001 C CNN
-F 1 "+12V" H 4665 5123 50  0000 C CNN
-F 2 "" H 4650 4950 50  0001 C CNN
-F 3 "" H 4650 4950 50  0001 C CNN
-	1    4650 4950
-	1    0    0    -1
-$EndComp
-$Comp
-L power:+5V #PWR?
-U 1 1 5EEA8FCB
-P 4800 5150
-F 0 "#PWR?" H 4800 5000 50  0001 C CNN
-F 1 "+5V" H 4815 5323 50  0000 C CNN
-F 2 "" H 4800 5150 50  0001 C CNN
-F 3 "" H 4800 5150 50  0001 C CNN
-	1    4800 5150
-	1    0    0    -1
-$EndComp
-$Comp
-L power:+3.3V #PWR?
-U 1 1 5EEA9354
-P 4950 5350
-F 0 "#PWR?" H 4950 5200 50  0001 C CNN
-F 1 "+3.3V" H 4965 5523 50  0000 C CNN
-F 2 "" H 4950 5350 50  0001 C CNN
-F 3 "" H 4950 5350 50  0001 C CNN
-	1    4950 5350
-	1    0    0    -1
-$EndComp
-$Comp
-L power:GND #PWR?
-U 1 1 5EEA957B
-P 4450 5500
-F 0 "#PWR?" H 4450 5250 50  0001 C CNN
-F 1 "GND" H 4455 5327 50  0000 C CNN
-F 2 "" H 4450 5500 50  0001 C CNN
-F 3 "" H 4450 5500 50  0001 C CNN
-	1    4450 5500
-	1    0    0    -1
-$EndComp
-$Comp
-L power:GNDA #PWR?
-U 1 1 5EEA98B3
-P 2750 4850
-F 0 "#PWR?" H 2750 4600 50  0001 C CNN
-F 1 "GNDA" H 2755 4677 50  0000 C CNN
-F 2 "" H 2750 4850 50  0001 C CNN
-F 3 "" H 2750 4850 50  0001 C CNN
-	1    2750 4850
-	1    0    0    -1
-$EndComp
-Wire Wire Line
-	3750 4600 2750 4600
-Wire Wire Line
-	2750 4600 2750 4800
-Wire Wire Line
-	3750 4800 2750 4800
-Connection ~ 2750 4800
-Wire Wire Line
-	2750 4800 2750 4850
-$Comp
-L power:GNDA #PWR?
-U 1 1 5EEABE68
-P 5100 4750
-F 0 "#PWR?" H 5100 4500 50  0001 C CNN
-F 1 "GNDA" H 5105 4577 50  0000 C CNN
-F 2 "" H 5100 4750 50  0001 C CNN
-F 3 "" H 5100 4750 50  0001 C CNN
-	1    5100 4750
-	1    0    0    -1
-$EndComp
-Wire Wire Line
-	5100 4750 5100 4700
-Wire Wire Line
-	5100 4500 4250 4500
-Wire Wire Line
-	4250 4700 5100 4700
-Connection ~ 5100 4700
-Wire Wire Line
-	5100 4700 5100 4500
-Wire Wire Line
-	4250 4800 4450 4800
-Wire Wire Line
-	4450 4800 4450 4900
-Wire Wire Line
-	4250 4900 4450 4900
-Connection ~ 4450 4900
-Wire Wire Line
-	4450 4900 4450 5100
-Wire Wire Line
-	4250 5100 4450 5100
-Connection ~ 4450 5100
-Wire Wire Line
-	4450 5100 4450 5300
-Wire Wire Line
-	4250 5300 4450 5300
-Connection ~ 4450 5300
-Wire Wire Line
-	4450 5300 4450 5500
-Wire Wire Line
-	4250 5400 4950 5400
-Wire Wire Line
-	4950 5400 4950 5350
-Wire Wire Line
-	4250 5200 4800 5200
-Wire Wire Line
-	4800 5200 4800 5150
-Wire Wire Line
-	4250 5000 4650 5000
-Wire Wire Line
-	4650 5000 4650 4950
-Wire Wire Line
-	4250 4600 4900 4600
-Wire Wire Line
-	3750 4500 3100 4500
-Wire Wire Line
-	3750 4700 3100 4700
-Wire Wire Line
-	3100 4900 3750 4900
-Wire Wire Line
-	3750 5000 3100 5000
-Wire Wire Line
-	3100 5100 3750 5100
-Wire Wire Line
-	3750 5200 3100 5200
-Wire Wire Line
-	3100 5300 3750 5300
-Wire Wire Line
-	3750 5400 3100 5400
-NoConn ~ 3650 2550
-NoConn ~ 4150 2550
-NoConn ~ 4150 2750
-NoConn ~ 3650 2750
-$Comp
-L Relay:G5LE-1 K?
-U 1 1 5EEBE0CB
-P 8000 3800
-F 0 "K?" H 8430 3846 50  0000 L CNN
-F 1 "G5LE-1" H 8430 3755 50  0000 L CNN
-F 2 "Relay_THT:Relay_SPDT_Omron-G5LE-1" H 8450 3750 50  0001 L CNN
-F 3 "http://www.omron.com/ecb/products/pdf/en-g5le.pdf" H 8000 3800 50  0001 C CNN
-	1    8000 3800
-	1    0    0    -1
-$EndComp
+$Sheet
+S 5350 1000 1800 1550
+U 5ED5374F
+F0 "ProbadorDriver" 118
+F1 "ProbadorDriver.sch" 118
+$EndSheet
+$Sheet
+S 8350 1100 1800 1700
+U 5ED538D0
+F0 "ProbadorTemporizador" 118
+F1 "ProbadorTemporizador.sch" 118
+$EndSheet
 $EndSCHEMATC
